File: nfc_card.kicad_pcb (KiCad board)
At the start: 2 copper layers, 2 parts, among them U1 ST25DV04K-JFR6D3

Commit message: stufffff
Parts:
- added U2: NFC_ANTENNA, Library:NFC_ANT, F.Cu at (154.7, 104.1)
- moved C1 15.4 mm to (152.0, 105.0)
- moved U1 15.4 mm to (151.0, 102.8)
Connections:
- U1 pad 5: Net-(U1-AC0) -> Net-(U1-AC1)
Routing:
- net Net-(U1-AC0): track 177.8 -> 2.82 mm, vias 2 -> 0
- net Net-(U1-AC1): track 0.00 -> 2.64 mm
Other:
- board outline added: 85.5 x 54 mm

Commit message: bit of design, needs to be finished
Parts:
- added G***: LOGO, LOGO, F.Cu at (112.0, 104.0)
- moved U1 2.70 mm to (152.5, 100.5)
- moved C1 2.06 mm to (152.5, 103.0)
Routing:
- net Net-(U1-AC1): track 2.64 -> 5.07 mm
- net Net-(U1-AC0): track 2.82 -> 4.44 mm
- net Net-(U1-VSS): track 2.69 -> 1.78 mm
- net Net-(U1-VCC): track 4.77 -> 5.56 mm
Other:
- outline, holes or cut-outs redrawn
- board text added: "- developer - 3d printer nerd - onboard reviewer - frc 1360"
- board text added: "blaze"
- board text added: "blazecoding.xyz or just tap your phone!"

Commit message: graphics!
Parts:
- added G***: LOGO, LOGO, F.Cu at (131.0, 116.5)
- added G***: LOGO, LOGO, F.Cu at (151.0, 121.5)
- added G***: LOGO, LOGO, F.Cu at (88.5, 92.0)
- added G***: LOGO, LOGO, F.Cu at (111.0, 100.0)

Commit message: almost done, one more session to go
Parts:
- added D1: LED, LED_SMD:LED_0201_0603Metric, F.Cu at (108.7, 82.5)
- added R1: 47ohm, Resistor_SMD:R_0201_0603Metric, F.Cu at (107.0, 82.5)
- U1: value ST25DV04K-JFR6D3 -> NT3H2111W0FHKH; footprint Package_DFN_QFN:ST_UFDFPN-12-1EP_3x3mm_P0.5mm_EP1.4x2.55mm -> Library:QFN8P50_160X160X50L40X20N
- U2: footprint Library:NFC_ANT -> Library:25X48MM_NFC_ANTENNA
- moved C1 48.8 mm to (107.8, 83.6), turned to 0 degrees
- moved U1 47.2 mm to (107.8, 85.6), turned to 180 degrees
- moved U2 40.2 mm to (114.5, 104.5), turned to 0 degrees
Connections:
- C1 pad 2: Net-(U1-VSS) -> Net-(D1-K)
- U1 pad 1: unconnected-(U1-LPD-Pad1) -> Net-(U1-LA)
- U1 pad 2: unconnected-(U1-NC-Pad2) -> Net-(D1-K)
- U1 pad 4: Net-(U1-AC0) -> unconnected-(U1-FD-Pad4)
- U1 pad 5: Net-(U1-AC1) -> unconnected-(U1-SDA-Pad5)
- U1 pad 6: Net-(U1-VSS) -> Net-(U1-VCC)
- U1 pad 7: unconnected-(U1-SDA-Pad7) -> Net-(U1-VCC)
- U1 pad 8: unconnected-(U1-SCL-Pad8) -> Net-(U1-LB)
- U2 pad P$2: (no net) -> Net-(U1-LB)
Routing:
- net Net-(U1-LB): track 0.00 -> 12.2 mm, vias 0 -> 1
- net Net-(U1-LA): track 0.00 -> 7.30 mm
- net Net-(U1-AC1): track 5.07 -> 0.00 mm
- net Net-(D1-K): track 0.00 -> 4.66 mm
- net Net-(U1-AC0): track 4.44 -> 0.00 mm
- net Net-(U1-VSS): track 1.78 -> 0.00 mm
- net Net-(D1-A): track 0.00 -> 1.02 mm
